File: devboard/devboard.kicad_sch (KiCad schematic)
At the start: 0 parts

Commit message: changes
Parts:
- added C1, C10: 1uF, symbol Device:C
- added C11, C12, C2, C3, C4, C5, C6, C7, C8, C9: 0.1uF, symbol Device:C
- added C13, C14: 10uF, symbol Device:C
- added J1: USB_C_Receptacle_USB2.0_14P, symbol Connector:USB_C_Receptacle_USB2.0_14P
- added R1, R2: 5.1K, symbol Device:R
- added R3, R4: 27, symbol Device:R
- added U1: RP2040, Package_DFN_QFN:QFN-56-1EP_7x7mm_P0.4mm_EP3.2x3.2mm, symbol MCU_RaspberryPi:RP2040
- added U2: NCP1117-3.3_SOT223, Package_TO_SOT_SMD:SOT-223-3_TabPin2, symbol Regulator_Linear:NCP1117-3.3_SOT223
- added Y1: Crystal_GND24, symbol Device:Crystal_GND24
Connections:
- new net: J1.A5 (CC1), R1.1
- new net: R4.2, U1.47 (USB_DP)
- new net: R3.2, U1.46 (USB_DM)
- new net: Y1.2 (G), Y1.4 (G)
- new net: J1.B5 (CC2), R2.1
- new net +1V1: C10.1, C11.1, C12.1, U1.43 (ADC_AVDD), U1.48 (USB_VDD)
- new net +3V3: C1.1, C14.1, C2.1, C3.1, C4.1, C5.1, C6.1, C7.1, C8.1, C9.1, U1.1 (IOVDD), U1.10 (IOVDD), U1.22 (IOVDD), U1.23 (DVDD), U1.33 (IOVDD), U1.42 (IOVDD), U1.44 (VREG_VIN), U1.45 (VREG_VOUT), U1.49 (IOVDD), U1.50 (DVDD), U2.2 (VO)
- new net GND: C1.2, C10.2, C11.2, C12.2, C13.2, C14.2, C2.2, C3.2, C4.2, C5.2, C6.2, C7.2, C8.2, C9.2, J1.A1 (GND), J1.A12 (GND), J1.B1 (GND), J1.B12 (GND), J1.S1 (SHIELD), R1.2, R2.2, U1.57 (GND), U2.1 (GND)
- new net USB_D+: J1.A6 (D+), J1.B6 (D+), R4.1
- new net USB_D-: J1.A7 (D-), J1.B7 (D-), R3.1
- new net VBUS: C13.1, J1.A4 (VBUS), J1.A9 (VBUS), J1.B4 (VBUS), J1.B9 (VBUS), U2.3 (VI)
- new net XIN: U1.20 (XIN)
- new net XOUT: U1.21 (XOUT)

Commit message: idk
Parts:
- removed Y1: Crystal_GND24, symbol Device:Crystal_GND24
- added C15: 10uF, symbol Device:C
Changed lines of the file:
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@@
 	)
 	(symbol
-		(lib_id "Device:Crystal_GND24")
-		(at 226.06 99.06 0)
+		(lib_id "Device:C")
+		(at 214.63 99.06 0)
 		(unit 1)
 		(exclude_from_sim no)
@@
 		(on_board yes)
 		(dnp no)
-		(fields_autoplaced yes)
-		(property "Reference" "Y1"
-			(at 226.06 90.17 0)
+		(property "Reference" "C15"
+			(at 214.63 97.282 0)
 			(effects
 				(font
 					(size 1.27 1.27)
 				)
+				(justify left)
 			)
 		)
-		(property "Value" "Crystal_GND24"
-			(at 226.06 92.71 0)
+		(property "Value" "10uF"
+			(at 214.63 101.092 0)
 			(effects
 				(font
 					(size 1.27 1.27)
 				)
+				(justify left)
 			)
 		)
 		(property "Footprint" ""
-			(at 226.06 99.06 0)
+			(at 215.5952 102.87 0)
 			(effects
 				(font
@@
 		)
 		(property "Datasheet" "~"
-			(at 226.06 99.06 0)
+			(at 214.63 99.06 0)
 			(effects
 				(font
@@
 			)
 		)
-		(property "Description" "Four pin crystal, GND on pins 2 and 4"
-			(at 226.06 99.06 0)
-			(effects
-				(font
-					(size 1.27 1.27)
-				)
-				(hide yes)
-			)
-		)
-		(property private "KLC_S3.3" "The rectangle is not a symbol body but a graphical element"
-			(at 226.06 111.76 0)
-			(show_name yes)
-			(effects
-				(font
-					(size 1.27 1.27)
-				)
-				(hide yes)
-			)
-		)
-		(property private "KLC_S4.1" "Some pins are on 50mil grid to make the symbol small"
-			(at 226.06 114.3 0)
-			(show_name yes)
+		(property "Description" "Unpolarized capacitor"
+			(at 214.63 99.06 0)
 			(effects
 				(font
@@
 		(pin "2"
 		)
-		(pin "4"
-		)
-		(pin "3"
-		)
 		(instances
-			(project ""
+			(project "devboard"
 				(path "/d109a607-c9d7-4c8e-a2b9-07e3c74c8bd3"
-					(reference "Y1")
+					(reference "C15")
 					(unit 1)
 				)
