File: devboard/devboard.kicad_sch (KiCad schematic)
At the start: 33 parts, among them J1 USB_C_Receptacle_USB2.0_14P, J2 Conn_01x20, J3 Conn_01x20, J4 Conn_01x03, SW1 SW_Push, U1 RP2040, U2 MCP1700x-120xxTT, U3 W25Q128JVS, Y1 ASCO

Commit message: Production file generation + final pcb update
Parts:
- C13, C14: footprint Capacitor_SMD:C_0201_0603Metric -> Capacitor_SMD:C_0603_1608Metric
- Y1: value ASCO -> 12MHz

Commit message: final fr
Other:
- note added: "Decoupling Capacitors"
- note added: "Flash Memory"
- note added: "LDO"
- note added: "Pin Layout"
- note added: "RP2040 Microcontroller"
- note added: "USB C"
- moved on the sheet: C1, C10, C11, C12, C2, C3, C4, C5, C6, C7, C8, C9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
