File: devboard/devboard.kicad_pcb (KiCad board)
At the start: 2 copper layers, 21 x 51 mm, 33 parts, among them J1 USB_C_Receptacle_USB2.0_14P, J2 Conn_01x20, J3 Conn_01x20, J4 Conn_01x03, SW1 SW_Push, U1 RP2040, U2 NCP1117-3.3_SOT223, U3 W25Q128JVS, Y1 ASCO

Commit message: PCB routing and changes
Parts:
- U2: value NCP1117-3.3_SOT223 -> MCP1700x-120xxTT; footprint Package_TO_SOT_SMD:SOT-223-3_TabPin2 -> Package_TO_SOT_SMD:SOT-23
- U3: footprint Package_SO:SOIC-8_5.3x5.3mm_P1.27mm -> Package_SON:Winbond_USON-8-1EP_3x2mm_P0.5mm_EP0.2x1.6mm
- moved C2 65.0 mm to (165.2, 74.0)
- moved R3 64.1 mm to (161.9, 66.7), turned to -90 degrees
- moved R4 63.1 mm to (160.9, 66.7), turned to -90 degrees
- moved C8 62.9 mm to (165.2, 77.8)
- moved C7 62.9 mm to (165.2, 75.8)
- moved C9 62.3 mm to (165.2, 76.8)
- moved C11 61.6 mm to (165.2, 73.0)
- moved C4 61.0 mm to (160.5, 81.4), turned to -90 degrees
- moved C10 60.6 mm to (164.2, 72.0)
- moved C12 59.2 mm to (162.8, 71.0), turned to 90 degrees
- moved C16 58.8 mm to (162.2, 84.2), turned to -90 degrees
- moved C1 55.4 mm to (155.3, 72.8), turned to 180 degrees
- moved C3 55.0 mm to (154.9, 76.9), turned to 180 degrees
- moved C13 54.8 mm to (157.0, 55.0), turned to 180 degrees
- moved C5 54.6 mm to (154.9, 77.9), turned to 180 degrees
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Connections:
- C16 pad 1: Net-(Y1-GND) -> Net-(Y1-Tri-State)
- R5 pad 1: Net-(Y1-GND) -> Net-(Y1-Tri-State)
- Y1 pad 1: GND -> Net-(Y1-Tri-State)
- Y1 pad 2: Net-(Y1-GND) -> GND
- Y1 pad 3: GND -> XIN
- Y1 pad 4: XIN -> GND
Routing:
- net QSPI_SS: track 0.00 -> 7.41 mm
- net QSPI_SD1: track 0.00 -> 6.70 mm
- net QSPI_SD2: track 0.00 -> 5.39 mm
- net QSPI_SD3: track 0.00 -> 5.24 mm
- net QSPI_SCLK: track 0.00 -> 4.54 mm
- net QSPI_SD0: track 0.00 -> 3.60 mm
- net USB_D+: track 0.00 -> 3.06 mm
- net USB_D-: track 0.00 -> 2.99 mm

Commit message: Production file generation + final pcb update
Parts:
- C13, C14: footprint Capacitor_SMD:C_0201_0603Metric -> Capacitor_SMD:C_0603_1608Metric
- Y1: value ASCO -> 12MHz
- moved J3 48.3 mm to (168.9, 96.4), turned to 180 degrees
- moved R1 45.3 mm to (162.2, 55.1)
- moved R2 42.1 mm to (158.9, 55.0)
- moved R5 40.1 mm to (160.2, 81.4), turned to 90 degrees
- moved SW1 30.1 mm to (156.8, 63.8), turned to 180 degrees
- moved R7 19.1 mm to (155.8, 72.3), turned to -90 degrees
- moved R6 16.6 mm to (154.5, 66.5), turned to -90 degrees
- moved C5 12.6 mm to (165.3, 70.8), turned to 0 degrees
- moved C4 12.6 mm to (165.3, 69.8), turned to 0 degrees
- moved C6 11.9 mm to (165.3, 68.8), turned to 0 degrees
- moved C8 11.6 mm to (160.5, 67.2)
- moved C9 11.6 mm to (160.5, 66.2)
- moved C3 9.54 mm to (160.5, 69.2), turned to 0 degrees
- moved C1 6.93 mm to (160.5, 68.2), turned to 0 degrees
- moved R3 4.33 mm to (161.8, 71.0)
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Routing:
- net +3V3: track 0.00 -> 51.5 mm, vias 0 -> 4
- net GPIO0: track 0.00 -> 32.4 mm, vias 0 -> 1
- net GPIO1: track 0.00 -> 29.0 mm, vias 0 -> 1
- net GPIO29_ADC3: track 0.00 -> 26.1 mm, vias 0 -> 1
- net GPIO2: track 0.00 -> 23.5 mm, vias 0 -> 1
- net GPIO28_ADC2: track 0.00 -> 21.8 mm, vias 0 -> 1
- net GPIO15: track 0.00 -> 21.0 mm
- net VBUS: track 0.00 -> 21.0 mm
- net SWDI0: track 0.00 -> 20.3 mm, vias 0 -> 1
- net GPIO3: track 0.00 -> 19.6 mm
- net GPIO16: track 0.00 -> 19.5 mm
- net GPIO4: track 0.00 -> 19.3 mm, vias 0 -> 1
- net USB_D-: track 2.99 -> 21.9 mm
- net USB_D+: track 3.06 -> 22.0 mm
- net GPIO14: track 0.00 -> 18.3 mm
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- added copper zone on B.Cu, net GND
- added copper zone on F.Cu, net GND

Commit message: final fr
Parts:
- moved C9 15.2 mm to (161.2, 81.4), turned to -90 degrees
- moved C8 15.2 mm to (162.2, 82.3), turned to -90 degrees
- moved C5 12.5 mm to (154.5, 77.2), turned to 180 degrees
- moved C6 11.1 mm to (154.8, 72.3), turned to 90 degrees
- moved C4 7.80 mm to (166.2, 77.5)
- moved C7 0.17 mm to (165.1, 71.8)
- moved C10 0.16 mm to (163.2, 71.6)
- moved C11 0.16 mm to (163.2, 69.6)
- moved C12 0.16 mm to (163.2, 70.6)
- moved C2 0.15 mm to (164.8, 72.8)
- turned C15 to 90 degrees
Routing:
- net GND: track 8.77 -> 21.3 mm, vias 6 -> 8
- net +3V3: track 51.5 -> 56.6 mm
- net SWCLK: track 17.3 -> 20.0 mm, vias 0 -> 2
- net GPIO8: track 7.16 -> 8.19 mm
- net SWDI0: track 20.3 -> 19.8 mm, vias 1 -> 0
